File: Asotin.sch (KiCad schematic (older format))
At the start: 2 parts

Commit message: add keebio library
Parts:
- added C1, C2, C5: .1uF, Capacitor_SMD:C_0805_2012Metric, symbol Device:C_Small
- added C3, C4: 22pF, Capacitor_SMD:C_0805_2012Metric, symbol Device:C_Small
- added C6: 10uF, Capacitor_SMD:C_0805_2012Metric, symbol Device:C_Small
- added C7: 1uF, Capacitor_SMD:C_0805_2012Metric, symbol Device:C_Small
- added D1, D2, D3, D4: SOD-123, Diode_SMD:D_SOD-123, symbol Device:D_Small
- added D13: SR05, Diode_SMD:D_SOD-123, symbol Power_Protection:PRTR5V0U2X
- added J1: USB_C_Receptacle_USB2.0, symbol Connector:USB_C_Receptacle_USB2.0
- added MX1, MX2, MX3, MX4: MX-NoLED, symbol MX_Alps_Hybrid:MX-NoLED
- added R1, R2: 22, symbol Device:R_Small
- added R3: 10k, symbol Device:R_Small
- added SW1: SW_Push, symbol Switch:SW_Push
- added Y1: 16MHz, symbol Device:Crystal_GND24_Small
- gave numbers to parts that had none: 2
Connections:
- net +5V: now also U1.7 (VBUS), C1.1, C2.1, C5.1, C6.1, R3.2
- net GND: now also C1.2, C2.2, C3.2, C4.2, C5.2, C6.2, C7.2, D13.1 (GND), J1.A1 (GND), J1.A12 (GND), J1.B1 (GND), J1.B12 (GND), SW1.1, Y1.2, Y1.4
- net at U1.13 (~RESET): now also R3.1, SW1.2
- net at U1.16 (XTAL2): now also C4.1, Y1.3
- net at U1.17 (XTAL1): now also C3.1, Y1.1
- net at U1.3 (D-): now also R1.1
- net at U1.4 (D+): now also R2.1
- net at U1.6 (UCAP): now also C7.1
- new net: D1.2 (A), MX1.2 (ROW)
- new net: D3.2 (A), MX3.2 (ROW)
- new net: D2.2 (A), MX2.2 (ROW)
- new net: D4.2 (A), MX4.2 (ROW)
- new net COL0: MX1.1 (COL), MX2.1 (COL)
- new net COL1: MX3.1 (COL), MX4.1 (COL)
- new net D+: D13.3 (I/O2), J1.A6 (D+), J1.B6 (D+), R2.2
- new net D-: D13.2 (I/O1), J1.A7 (D-), J1.B7 (D-), R1.2
- new net ROW0: D1.1 (K), D3.1 (K)
- new net ROW1: D2.1 (K), D4.1 (K)
- new net VCC: D13.4 (VCC), J1.A4 (VBUS), J1.A9 (VBUS), J1.B4 (VBUS), J1.B9 (VBUS)
